File: circuits/pc-02_16bit_register/16bit_register.kicad_pcb (KiCad board)
At the start: 2 copper layers, 99.1 x 99.1 mm, 26 parts, among them U1 74HC273, U2 74HC273, U3 74HC244, U4 74HC244, U5 74HC244, U6 74HC244

Commit message: pc-02: move decoder hardware onto board
Parts:
- removed R10, R11, R12, R13: 100k, Resistor_SMD:R_0603_1608Metric
- added U10: 4071, Package_DIP:DIP-14_W7.62mm_LongPads, F.Cu at (78.7, 109.9)
- added U12: 4011, Package_DIP:DIP-14_W7.62mm_LongPads, F.Cu at (51.4, 66.7)
- added U7: 74HC138, Package_DIP:DIP-16_W7.62mm_LongPads, F.Cu at (52.7, 93.3)
- added U8: 4011, Package_DIP:DIP-14_W7.62mm_LongPads, F.Cu at (109.2, 109.9)
- added U9: 4071, Package_DIP:DIP-14_W7.62mm_LongPads, F.Cu at (94.0, 109.9)
- R1, R2, R3, R4, R5, R7, R8, R9: value 0R -> R
- moved R4 53.9 mm to (52.7, 86.4), turned to -90 degrees
- moved R3 50.1 mm to (55.2, 86.4), turned to -90 degrees
- moved R2 46.7 mm to (57.8, 86.4), turned to -90 degrees
- moved R1 42.7 mm to (60.3, 86.4), turned to -90 degrees
- moved R7 12.0 mm to (115.6, 105.4), turned to 0 degrees
- moved R9 9.75 mm to (115.6, 98.4), turned to 0 degrees
- moved R8 9.58 mm to (115.6, 95.2), turned to 0 degrees
- moved R5 8.01 mm to (115.6, 102.2), turned to 0 degrees
Connections:
- CTRL_BUS1 pad 1: /~{readPC_low} -> /data_source0
- CTRL_BUS1 pad 10: unconnected-(CTRL_BUS1-Pin_10-Pad10) -> /action1
- CTRL_BUS1 pad 11: unconnected-(CTRL_BUS1-Pin_11-Pad11) -> /action2
- CTRL_BUS1 pad 12: unconnected-(CTRL_BUS1-Pin_12-Pad12) -> /action3
- CTRL_BUS1 pad 13: unconnected-(CTRL_BUS1-Pin_13-Pad13) -> /action4
- CTRL_BUS1 pad 14: unconnected-(CTRL_BUS1-Pin_14-Pad14) -> /adr_source0
- CTRL_BUS1 pad 15: unconnected-(CTRL_BUS1-Pin_15-Pad15) -> /adr_source1
- CTRL_BUS1 pad 16: unconnected-(CTRL_BUS1-Pin_16-Pad16) -> /adr_source2
- CTRL_BUS1 pad 2: /~{readPC_high} -> /data_source1
- CTRL_BUS1 pad 3: /~{readSP_low} -> /data_source2
- CTRL_BUS1 pad 4: /~{readSP_high} -> /data_source3
- CTRL_BUS1 pad 5: /~{readPC} -> /data_target0
- CTRL_BUS1 pad 6: /~{readSP} -> /data_target1
- CTRL_BUS1 pad 7: /writePC -> /data_target2
- CTRL_BUS1 pad 8: /writeSP -> /write
- CTRL_BUS1 pad 9: unconnected-(CTRL_BUS1-Pin_9-Pad9) -> /action0
- R1 pad 1: /~{readPC} -> /~{read8low}
- R1 pad 2: /read16 -> /~{r8_pcl}
- R2 pad 1: /~{readSP} -> /~{read8high}
- R2 pad 2: /read16 -> /~{r8_pch}
- R3 pad 1: /writePC -> /~{read8low}
- R3 pad 2: /write16 -> /~{r8_spl}
- R4 pad 1: /writeSP -> /~{read8high}
- R4 pad 2: /write16 -> /~{r8_sph}
- R5 pad 1: /~{readPC_low} -> Net-(R5-Pad1)
- R5 pad 2: /~{read8low} -> Net-(R5-Pad2)
- R7 pad 1: /~{readPC_high} -> /adr_source0
- R7 pad 2: /~{read8high} -> Net-(R5-Pad2)
- R8 pad 1: /~{readSP_low} -> Net-(R8-Pad1)
- R8 pad 2: /~{read8low} -> Net-(R8-Pad2)
- R9 pad 1: /~{readSP_high} -> /action0
- R9 pad 2: /~{read8high} -> Net-(R8-Pad2)
Routing:
- net /data_source0: track 0.00 -> 138.7 mm
- net /data_source1: track 0.00 -> 129.1 mm
- net /data_source2: track 0.00 -> 126.4 mm
- net VCC: track 157.0 -> 272.9 mm, vias 1 -> 0
- net /data_source3: track 0.00 -> 112.5 mm
- net /write: track 0.00 -> 100.8 mm, vias 0 -> 2
- net /action1: track 0.00 -> 68.9 mm
- net /action2: track 0.00 -> 58.6 mm
- net /read16: track 144.4 -> 88.9 mm, vias 1 -> 2
- net Net-(R8-Pad2): track 0.00 -> 54.1 mm, vias 0 -> 1
- net /adr_source2: track 0.00 -> 52.8 mm, vias 0 -> 1
- net /~{read8high}: track 97.5 -> 46.3 mm, vias 3 -> 0
- net /write16: track 58.1 -> 105.4 mm
- net /action3: track 0.00 -> 45.5 mm
- net Net-(R5-Pad2): track 0.00 -> 42.7 mm
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Other:
- board text added: "4011 (NAND)"
- board text added: "4071 (IOR)"
- board text added: "74138 (3-8 DECODER)"
