File: circuits/pc-02_16bit_register/16bit_register.kicad_sch (KiCad schematic)
At the start: 26 parts, among them U1 74HC273, U2 74HC273, U3 74HC244, U4 74HC244, U5 74HC244, U6 74HC244

Commit message: pc-02: move decoder hardware onto board
Parts:
- removed R10, R11, R12, R13: 100k, Resistor_SMD:R_0603_1608Metric, symbol Device:R
- added U10, U9: 4071, Package_DIP:DIP-14_W7.62mm_LongPads, symbol 4xxx:4071
- added U12, U8: 4011, Package_DIP:DIP-14_W7.62mm_LongPads, symbol 4xxx:4011
- added U7: 74HC138, Package_DIP:DIP-16_W7.62mm_LongPads, symbol 74xx:74HC138
- R1, R2, R3, R4, R5, R7, R8, R9: value 0R -> R
Connections:
- net GND: now also U10.5, U10.6, U10.7 (VSS), U10.8, U10.9, U12.12, U12.13, U12.7 (VSS), U7.4 (~{E0}), U7.5 (~{E1}), U7.8 (GND), U8.7 (VSS), U9.7 (VSS)
- net VCC: now also U10.14 (VDD), U12.14 (VDD), U7.16 (VCC), U8.14 (VDD), U9.14 (VDD)
- net read16: now also U9.10; no longer R1.2, R2.2
- net write16: now also U12.4; no longer R3.2, R4.2
- net ~{read8high}: now also R2.1, R4.1; no longer R7.2, R9.2
- net ~{read8low}: now also R1.1, R3.1; no longer R5.2, R8.2
- net action1: now reaches CTRL_BUS1.10 (Pin_10)
- net action1: now also U9.6
- net action2: now reaches CTRL_BUS1.11 (Pin_11)
- net action2: now also U9.2
- net action3: now reaches CTRL_BUS1.12 (Pin_12)
- net action3: now also U9.1
- net action4: now reaches CTRL_BUS1.13 (Pin_13)
- net action4: now also U8.8, U8.9
- net adr_source0: now reaches CTRL_BUS1.14 (Pin_14)
- net adr_source0: now also R7.1, U8.1, U8.2
- net adr_source1: now reaches CTRL_BUS1.15 (Pin_15)
- net adr_source1: now also U8.12, U8.13
- net adr_source2: now reaches CTRL_BUS1.16 (Pin_16)
- net adr_source2: now also U9.12
- net action0: now reaches CTRL_BUS1.9 (Pin_9)
- net action0: now also R9.1, U8.5, U8.6
- net writePC renamed data_target2
- net data_target2: no longer R3.1
- net writeSP renamed write
- net write: now also U12.1; no longer R4.1
- net ~{readPC_high} renamed data_source1
- net data_source1: now also U7.2 (A1); no longer R7.1
- net ~{readPC_low}: no longer names the net of R5.1
- net ~{readPC_low}: now also U8.3; no longer CTRL_BUS1.1 (Pin_1)
- net ~{readPC} renamed data_target0
- net data_target0: no longer R1.1
- net ~{readSP_high} renamed data_source3
- net data_source3: now also U7.6 (E2); no longer R9.1
- net ~{readSP_low}: no longer names the net of R8.1
- net ~{readSP_low}: now also U8.4; no longer CTRL_BUS1.3 (Pin_3)
- net ~{readSP} renamed data_target1
- net data_target1: no longer R2.1
- new net: U10.1, U9.4
- new net: U10.2, U8.10
- new net: U10.12, U10.3
- new net: U9.11, U9.9
- new net: U8.11, U9.13
- new net: R8.2, R9.2, U10.13
- new net: U12.10, U12.2
- new net: U12.3, U12.5, U12.6
- new net: U9.3, U9.5
- new net: U10.11, U12.8, U12.9
- new net: R5.2, R7.2, U9.8
- new net data_source0: CTRL_BUS1.1 (Pin_1), U7.1 (A0)
- new net data_source2: CTRL_BUS1.3 (Pin_3), U7.3 (A2)
- new net ~{r8_pch}: R2.2, U7.14 (~{Y1})
- new net ~{r8_pcl}: R1.2, U7.15 (~{Y0})
- new net ~{r8_sph}: R4.2, U7.12 (~{Y3})
- new net ~{r8_spl}: R3.2, U7.13 (~{Y2})
- no-connect marks 3 -> 10
