File: circuits/pc-xx_memory_stack_template/memory_stack_template.kicad_sch (KiCad schematic)
At the start: 8 parts, among them J1 Conn_01x10

Commit message: Kicad upgrade to 9.0
Other:
- title: PC-01 Dual Register Unit -> PC-XX TEMPLATE
Changed lines of the file:
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@@
 (kicad_sch
-	(version 20231120)
+	(version 20250114)
 	(generator "eeschema")
-	(generator_version "8.0")
+	(generator_version "9.0")
 	(paper "A4")
 	(title_block
-		(title "PC-01 Dual Register Unit")
-		(date "2025-02-11")
+		(title "PC-XX TEMPLATE")
 		(rev "A")
 	)
@@
 	(label "adr14"
 		(at 250.19 147.32 0)
-		(fields_autoplaced yes)
 		(effects
 			(font
@@
 	(label "data3"
 		(at 254 30.48 0)
-		(fields_autoplaced yes)
 		(effects
 			(font
@@
 	(label "adr5"
 		(at 250.19 124.46 0)
-		(fields_autoplaced yes)
 		(effects
 			(font
@@
 	(label "adr13"
 		(at 250.19 144.78 0)
-		(fields_autoplaced yes)
 		(effects
 			(font
@@
 	(label "~{reset}"
 		(at 262.89 48.26 180)
-		(fields_autoplaced yes)
 		(effects
 			(font
@@
 	(label "adr11"
 		(at 250.19 139.7 0)
-		(fields_autoplaced yes)
 		(effects
 			(font
@@
 	(label "adr2"
 		(at 250.19 116.84 0)
-		(fields_autoplaced yes)
 		(effects
 			(font
@@
 	(label "adr6"
 		(at 250.19 127 0)
-		(fields_autoplaced yes)
 		(effects
 			(font
@@
 	(label "data5"
 		(at 254 35.56 0)
-		(fields_autoplaced yes)
 		(effects
 			(font
@@
 	(label "mem_write"
 		(at 262.89 45.72 180)
-		(fields_autoplaced yes)
 		(effects
 			(font
@@
 	(label "~{mem_read}"
 		(at 262.89 43.18 180)
-		(fields_autoplaced yes)
 		(effects
 			(font
@@
 	(label "adr12"
 		(at 250.19 142.24 0)
-		(fields_autoplaced yes)
 		(effects
 			(font
@@
 	(label "adr1"
 		(at 250.19 114.3 0)
-		(fields_autoplaced yes)
 		(effects
 			(font
@@
 	(label "data7"
 		(at 254 40.64 0)
-		(fields_autoplaced yes)
 		(effects
 			(font
@@
 	(label "data4"
 		(at 254 33.02 0)
-		(fields_autoplaced yes)
 		(effects
 			(font
@@
 	(label "adr[0..15]"
 		(at 247.65 101.6 0)
-		(fields_autoplaced yes)
 		(effects
 			(font
@@
 	(label "adr0"
 		(at 250.19 111.76 0)
-		(fields_autoplaced yes)
 		(effects
 			(font
@@
 	(label "adr7"
 		(at 250.19 129.54 0)
-		(fields_autoplaced yes)
 		(effects
 			(font
@@
 	(label "data2"
 		(at 254 27.94 0)
-		(fields_autoplaced yes)
 		(effects
 			(font
@@
 	(label "adr8"
 		(at 250.19 132.08 0)
-		(fields_autoplaced yes)
 		(effects
 			(font
@@
 	(label "clock"
 		(at 262.89 50.8 180)
-		(fields_autoplaced yes)
 		(effects
 			(font
@@
 	(label "adr15"
 		(at 250.19 149.86 0)
-		(fields_autoplaced yes)
 		(effects
 			(font
@@
 	(label "adr4"
 		(at 250.19 121.92 0)
-		(fields_autoplaced yes)
 		(effects
 			(font
@@
 	(label "adr10"
 		(at 250.19 137.16 0)
-		(fields_autoplaced yes)
 		(effects
 			(font
@@
 	(label "data[0..7]"
 		(at 251.46 16.51 0)
-		(fields_autoplaced yes)
 		(effects
 			(font
@@
 	(label "adr9"
 		(at 250.19 134.62 0)
-		(fields_autoplaced yes)
 		(effects
 			(font
@@
 	(label "data1"
 		(at 254 25.4 0)
-		(fields_autoplaced yes)
 		(effects
 			(font
@@
 	(label "data6"
 		(at 254 38.1 0)
-		(fields_autoplaced yes)
 		(effects
 			(font
@@
 	(label "adr3"
 		(at 250.19 119.38 0)
-		(fields_autoplaced yes)
 		(effects
 			(font
@@
 	(label "data0"
 		(at 254 22.86 0)
-		(fields_autoplaced yes)
 		(effects
 			(font
@@
 		)
 	)
+	(embedded_fonts no)
 )

Commit message: Update memory_stack_template.kicad_sch
Connections:
- net mem_write renamed ~{mem_write}
Changed lines of the file:
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@@
 		)
 	)
-	(label "mem_write"
+	(label "~{mem_write}"
 		(at 262.89 45.72 180)
 		(effects
