File: circuits/pc-06_alu_logic/alu_logic.kicad_pcb (KiCad board)
At the start: 2 copper layers, 99.1 x 99.1 mm, 20 parts, among them J1 Conn_01x10, U1 74HC244 driver1, U10 gatesB, U2 notL, U3 iorL, U4 primL, U5 74HC244 driver2, U6 gatesA, U7 notH, U8 iorH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

Commit message: add filter and decoupling capacitors to all boards
Parts:
- added C1: C_Polarized, Capacitor_SMD:CP_Elec_5x5.3, F.Cu at (61.9, 30.5)
- added C2: C, Capacitor_SMD:C_0603_1608Metric, F.Cu at (65.4, 57.8)
- added C3: C, Capacitor_SMD:C_0603_1608Metric, F.Cu at (102.2, 52.2)
- added C4: C, Capacitor_SMD:C_0603_1608Metric, F.Cu at (63.5, 68.1)
- added C5: C, Capacitor_SMD:C_0603_1608Metric, F.Cu at (93.3, 71.0)
- added C6: C, Capacitor_SMD:C_0603_1608Metric, F.Cu at (118.1, 87.5)
Routing:
- net VCC: track 301.0 -> 308.9 mm
