File: circuits/pc-09_orchestrator_interconnect/orchestrator_interconnect.kicad_pcb (KiCad board)
At the start: 2 copper layers, 99.1 x 99.1 mm, 14 parts, among them J4 Conn_01x08, J5 Conn_01x05, J6 Conn_01x07, U1 4078, U2 74HC74, U3 4011, U4 4081, U5 4081, U6 74HC138

Commit message: bus spy, mock orchestrator & cleanup
Other:
- board text added: "4011 (NAND)"
- board text added: "4078 (BUS NOR)"
- board text added: "4081 (AND)"
- board text added: "74138 (3-8 DECODER)"
- board text added: "7474 (D-FF)"
Changed lines of the file:
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@@
 		(layer "Edge.Cuts")
+	)
+	(gr_text "7474 (D-FF)"
+		(at 76.2 79.375 90)
+		(layer "F.SilkS")
+		(effects
+			(font
+				(size 1 1)
+				(thickness 0.1)
+			)
+		)
 	)
 	(gr_text "MAIN INTERLINK"
@@
 			)
 			(justify left bottom)
+		)
+	)
+	(gr_text "4078 (BUS NOR)"
+		(at 72.39 104.14 0)
+		(layer "F.SilkS")
+		(effects
+			(font
+				(size 1 1)
+				(thickness 0.1)
+			)
+		)
+	)
+	(gr_text "74138 (3-8 DECODER)"
+		(at 76.2 48.895 90)
+		(layer "F.SilkS")
+		(effects
+			(font
+				(size 1 1)
+				(thickness 0.1)
+			)
+		)
+	)
+	(gr_text "4081 (AND)"
+		(at 91.44 50.165 90)
+		(layer "F.SilkS")
+		(effects
+			(font
+				(size 1 1)
+				(thickness 0.1)
+			)
+		)
+	)
+	(gr_text "4011 (NAND)"
+		(at 106.68 50.165 90)
+		(layer "F.SilkS")
+		(effects
+			(font
+				(size 1 1)
+				(thickness 0.1)
+			)
 		)
 	)
@@
 		)
 	)
+	(gr_text "4081 (AND)"
+		(at 122.555 50.165 90)
+		(layer "F.SilkS")
+		(effects
+			(font
+				(size 1 1)
+				(thickness 0.1)
+			)
+		)
+	)

Commit message: add filter and decoupling capacitors to all boards
Parts:
- added C1: C_Polarized, Capacitor_SMD:CP_Elec_5x5.3, F.Cu at (54.0, 44.7)
- added C2: C, Capacitor_SMD:C_0603_1608Metric, F.Cu at (114.3, 41.8)
- added C3: C, Capacitor_SMD:C_0603_1608Metric, F.Cu at (79.2, 67.3)
- added C4: C, Capacitor_SMD:C_0603_1608Metric, F.Cu at (79.2, 112.4)
- added C5: C, Capacitor_SMD:C_0603_1608Metric, F.Cu at (79.2, 35.6)
- added C6: C, Capacitor_SMD:C_0603_1608Metric, F.Cu at (98.8, 39.6)
Routing:
- net VCC: track 250.4 -> 284.3 mm
- net Net-(U6-~{Y6}): track 50.7 -> 52.4 mm
- net GND: vias 0 -> 4
