File: circuits/pc-10_bus_spy/bus_spy.kicad_pcb (KiCad board)
At the start: 2 copper layers, 99.1 x 99.1 mm, 91 parts, among them Q1 2N7002, Q10 2N7002, Q11 2N7002, Q12 2N7002, Q13 2N7002, Q14 2N7002, Q15 2N7002, Q16 2N7002, Q17 2N7002, Q18 2N7002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

Commit message: add filter and decoupling capacitors to all boards
Parts:
- added C1: C_Polarized, Capacitor_SMD:CP_Elec_5x5.3, F.Cu at (62.2, 34.0)
Routing:
- net VCC: track 190.3 -> 200.4 mm
Other:
- board text added: "RESET"
