File: circuits/pc-xx_orchestrator_stack_template/orchestrator_stack_template.kicad_sch (KiCad schematic)
At the start: 8 parts

Commit message: microcode pcb
Connections:
- net continue: now also BACKPLANE2.13 (Pin_13); no longer BACKPLANE2.16 (Pin_16)
- net flag_c: now also BACKPLANE2.14 (Pin_14); no longer BACKPLANE2.13 (Pin_13)
- net flag_s: now also BACKPLANE2.16 (Pin_16); no longer BACKPLANE2.15 (Pin_15)
- net flag_z: now also BACKPLANE2.15 (Pin_15); no longer BACKPLANE2.14 (Pin_14)
- net ~{clock}: no longer names the net of BACKPLANE1.2 (Pin_2)
- no-connect marks 0 -> 3
Changed lines of the file:
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@@
 		(color 0 0 0 0)
+	)
+	(no_connect
+		(at 33.02 154.94)
+	)
+	(no_connect
+		(at 33.02 170.18)
+	)
+	(no_connect
+		(at 33.02 167.64)
 	)
 	(bus_entry
@@
 	(wire
 		(pts
+			(xy 39.37 157.48) (xy 33.02 157.48)
+		)
+		(stroke
+			(width 0)
+			(type default)
+		)
+	)
+	(wire
+		(pts
 			(xy 34.29 190.5) (xy 33.02 190.5)
 		)
@@
 		)
 	)
+	(wire
+		(pts
+			(xy 39.37 152.4) (xy 33.02 152.4)
+		)
+		(stroke
+			(width 0)
+			(type default)
+		)
+	)
 	(bus
 		(pts
@@
 	(wire
 		(pts
+			(xy 247.65 129.54) (xy 260.35 129.54)
+		)
+		(stroke
+			(width 0)
+			(type default)
+		)
+	)
+	(wire
+		(pts
 			(xy 254 35.56) (xy 262.89 35.56)
 		)
@@
 		(pts
 			(xy 254 38.1) (xy 262.89 38.1)
+		)
+		(stroke
+			(width 0)
+			(type default)
+		)
+	)
+	(wire
+		(pts
+			(xy 39.37 160.02) (xy 33.02 160.02)
 		)
 		(stroke
@@
 	)
 	(label "flag_s"
-		(at 33.02 106.68 0)
+		(at 33.02 109.22 0)
 		(effects
 			(font
@@
 		)
 	)
-	(label "~{reset}"
-		(at 33.02 157.48 0)
-		(effects
-			(font
-				(size 1.27 1.27)
-			)
-			(justify left bottom)
-		)
-	)
 	(label "data4"
 		(at 254 33.02 0)
@@
 	)
 	(label "flag_z"
-		(at 33.02 104.14 0)
+		(at 33.02 106.68 0)
 		(effects
 			(font
@@
 		)
 	)
-	(label "~{halt}"
-		(at 33.02 160.02 0)
-		(effects
-			(font
-				(size 1.27 1.27)
-			)
-			(justify left bottom)
-		)
-	)
-	(label "~{reset}"
-		(at 262.89 50.8 180)
-		(effects
-			(font
-				(size 1.27 1.27)
-			)
-			(justify right bottom)
-		)
-	)
 	(label "cmd_5"
 		(at 33.02 83.82 0)
@@
 		)
 	)
-	(label "clock"
-		(at 33.02 152.4 0)
-		(effects
-			(font
-				(size 1.27 1.27)
-			)
-			(justify left bottom)
-		)
-	)
 	(label "action_1"
 		(at 260.35 134.62 180)
@@
 		)
 	)
-	(label "clock"
-		(at 260.35 129.54 180)
-		(effects
-			(font
-				(size 1.27 1.27)
-			)
-			(justify right bottom)
-		)
-	)
 	(label "data6"
 		(at 254 38.1 0)
@@
 	)
 	(label "continue"
-		(at 33.02 109.22 0)
+		(at 33.02 101.6 0)
 		(effects
 			(font
@@
 	)
 	(label "flag_c"
-		(at 33.02 101.6 0)
+		(at 33.02 104.14 0)
 		(effects
 			(font
@@
 		)
 	)
-	(label "~{clock}"
-		(at 33.02 154.94 0)
-		(effects
-			(font
-				(size 1.27 1.27)
-			)
-			(justify left bottom)
-		)
-	)
+	(global_label "~{reset}"
+		(shape input)
+		(at 39.37 157.48 0)
+		(fields_autoplaced yes)
+		(effects
+			(font
+				(size 1.27 1.27)
+			)
+			(justify left)
+		)
+		(property "Intersheetrefs" "${INTERSHEET_REFS}"
+			(at 47.0724 157.48 0)
+			(effects
+				(font
+					(size 1.27 1.27)
+				)
+				(justify left)
+				(hide yes)
+			)
+		)
+	)
+	(global_label "~{halt}"
+		(shape input)
+		(at 39.37 160.02 0)
+		(fields_autoplaced yes)
+		(effects
+			(font
+				(size 1.27 1.27)
+			)
+			(justify left)
+		)
+		(property "Intersheetrefs" "${INTERSHEET_REFS}"
+			(at 46.0441 160.02 0)
+			(effects
+				(font
+					(size 1.27 1.27)
+				)
+				(justify left)
+				(hide yes)
+			)
+		)
+	)
+	(global_label "~{reset}"
+		(shape input)
+		(at 262.89 50.8 180)
+		(fields_autoplaced yes)
+		(effects
+			(font
+				(size 1.27 1.27)
+			)
+			(justify right)
+		)
+		(property "Intersheetrefs" "${INTERSHEET_REFS}"
+			(at 255.1876 50.8 0)
+			(effects
+				(font
+					(size 1.27 1.27)
+				)
+				(justify right)
+				(hide yes)
+			)
+		)
+	)
+	(global_label "clock"
+		(shape input)
+		(at 247.65 129.54 180)
+		(fields_autoplaced yes)
+		(effects
+			(font
+				(size 1.27 1.27)
+			)
+			(justify right)
+		)
+		(property "Intersheetrefs" "${INTERSHEET_REFS}"
+			(at 239.6453 129.54 0)
+			(effects
+				(font
+					(size 1.27 1.27)
+				)
+				(justify right)
+				(hide yes)
+			)
+		)
+	)
+	(global_label "clock"
+		(shape input)
+		(at 39.37 152.4 0)
+		(fields_autoplaced yes)
+		(effects
+			(font
+				(size 1.27 1.27)
+			)
+			(justify left)
+		)
+		(property "Intersheetrefs" "${INTERSHEET_REFS}"
+			(at 47.3747 152.4 0)
+			(effects
+				(font
+					(size 1.27 1.27)
+				)
+				(justify left)
+				(hide yes)
+			)
+		)
+	)
