File: circuits/pc-07_ram_unit/ram_unit.kicad_sch (KiCad schematic)
At the start: 12 parts, among them U5 74HC138, U6 4011

Commit message: pc-08: decoder unit
Parts:
- removed U6: 4011, Package_DIP:DIP-14_W7.62mm_LongPads, symbol 4xxx:4011
Connections:
- net ~{write_pulse} is gone; now on net ~{mem_write}: U1.27 (~{WE}), U2.27 (~{WE}), U3.27 (~{WE}), U4.27 (~{WE})
- net mem_write renamed ~{mem_write}
- no-connect marks 8 -> 5

Commit message: add filter and decoupling capacitors to all boards
Parts:
- added C1: C_Polarized, Capacitor_SMD:CP_Elec_5x5.3, symbol Device:C_Polarized
- added C2, C3, C4, C5, C6: C, Capacitor_SMD:C_0603_1608Metric, symbol Device:C
Connections:
- net GND: now also C1.2, C2.2, C3.2, C4.2, C5.2, C6.2
- net VCC: now also C1.1, C2.1, C3.1, C4.1, C5.1, C6.1

Commit message: PC-07: reworked RAM unit: falling edge of !mem_write signal is converted to a low-pulse.
In experiments, 2 ceramic caps of 100nF each in series, and 2 resistors of 150 ohms yielded pulse widths of a just a few microseconds at clock rates of up to 25 kHz.
Parts:
- added C7, C8: 100nF, Capacitor_SMD:C_0603_1608Metric, symbol Device:C
- added Q1, Q2: 2N7000, Package_TO_SOT_THT:TO-92_Inline, symbol Transistor_FET:2N7000
- added R1, R2: 150R, Resistor_SMD:R_0603_1608Metric, symbol Device:R
- added R3: 1k, Resistor_SMD:R_0603_1608Metric, symbol Device:R
- added U6: 4011, Package_DIP:DIP-14_W7.62mm_LongPads, symbol 4xxx:4011
Connections:
- net GND: now also Q1.1 (S), Q2.1 (S), U6.1, U6.2, U6.5, U6.6, U6.7 (VSS)
- net VCC: now also R1.1, R2.1, R3.1, U6.14 (VDD)
- net ~{mem_write}: now also U6.8, U6.9; no longer U1.27 (~{WE}), U2.27 (~{WE}), U3.27 (~{WE}), U4.27 (~{WE})
- new net: C7.2, C8.1
- new net: C8.2, Q2.2 (G), R2.2
- new net: Q2.3 (D), R3.2, U6.12, U6.13
- new net: C7.1, Q1.3 (D), R1.2
- new net: Q1.2 (G), U6.10
- new net ~{write_pulse}: U1.27 (~{WE}), U2.27 (~{WE}), U3.27 (~{WE}), U4.27 (~{WE}), U6.11
- no-connect marks 5 -> 7
Other:
- title: PC-XX TEMPLATE -> PC-07 RAM Module
- moved on the sheet: C1, C2, C3, C4, C5, C6, U5

Commit message: pcb design
Parts:
- removed U6: 4011, Package_DIP:DIP-14_W7.62mm_LongPads, symbol 4xxx:4011
- added U7: 74HC14, Package_DIP:DIP-14_W7.62mm, symbol 74xx:74HC14
- Q1, Q2: footprint Package_TO_SOT_THT:TO-92_Inline -> Package_TO_SOT_THT:TO-92_Inline_Wide
Connections:
- net GND: now also U7.1, U7.3, U7.5, U7.7 (GND), U7.9
- net VCC: now also U7.14 (VCC)
- net ~{mem_write}: now also U7.11
- net ~{write_pulse}: now also U7.12
- net at Q2.3 (D), R3.2: now also U7.13
- net at Q1.2 (G): now also U7.10
- no-connect marks 7 -> 9
