File: circuits/pc-08_command_decoder/command_decoder.kicad_pcb (KiCad board)
At the start: 2 copper layers, 99.1 x 99.1 mm, 34 parts, among them J1 Screw_Terminal_01x02, J2 Conn_01x05, J3 Conn_01x03, J4 Conn_01x08, J5 Conn_01x05, J6 Conn_01x07, U1 74HC138, U2 74HC138, U3 74HC138, U4 74HC138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

Commit message: update documentation and update PCBs for interrupts
Parts:
- J3: value Conn_01x03 -> Conn_01x01; footprint Connector_PinHeader_2.54mm:PinHeader_1x03_P2.54mm_Vertical -> Connector_PinHeader_2.54mm:PinHeader_1x01_P2.54mm_Vertical
- moved J3 9.71 mm to (123.8, 64.1), turned to 180 degrees
Connections:
- CTRL_BUS2 pad 13: unconnected-(CTRL_BUS2-Pin_13-Pad13) -> /~{readIPC_low}
- CTRL_BUS2 pad 14: unconnected-(CTRL_BUS2-Pin_14-Pad14) -> /~{readIPC_high}
- U2 pad 10: Net-(J3-Pin_2) -> /~{readIPC_high}
- U2 pad 11: Net-(J3-Pin_3) -> /~{readIPC_low}
- U6 pad 10: /writeALU -> unconnected-(U6-Pad10)
- U6 pad 11: unconnected-(U6-Pad11) -> /writeALU
- U6 pad 12: VCC -> /~{writeALU}
- U6 pad 13: VCC -> /~{writeALU}
- U6 pad 8: /~{writeALU} -> GND
- U6 pad 9: /~{writeALU} -> GND
Routing:
- net /~{readIPC_low}: track 0.00 -> 83.2 mm
- net /~{readIPC_high}: track 0.00 -> 77.9 mm
- net Net-(J3-Pin_3): track 19.0 -> 0.00 mm
- net /writeALU: track 109.1 -> 90.4 mm
- net Net-(J3-Pin_2): track 15.8 -> 0.00 mm
- net /~{writeALU}: track 46.0 -> 38.0 mm
- net Net-(J3-Pin_1): track 22.5 -> 15.7 mm
- net GND: track 335.8 -> 329.5 mm, vias 8 -> 9
- net /~{readSP}: track 92.6 -> 90.0 mm
- net /~{readPC}: track 81.4 -> 78.8 mm
- net /~{writeL1}: track 18.1 -> 20.0 mm
- net /~{adrL}: track 80.1 -> 78.3 mm
- net /~{adrCD}: track 82.3 -> 80.4 mm
- net /~{readPC_low}: track 79.4 -> 77.9 mm
- net /~{readALU}: track 52.2 -> 51.1 mm
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Other:
- board text added: "~{DSRC 7}"
- board text removed: "12 13 7"
- board text removed: "~{DSRC}"
