File: circuits/pc-13_microcode/microcode.kicad_pcb (KiCad board)
At the start: 2 copper layers, 99.1 x 99.1 mm, 12 parts, among them J1 Conn_01x05, U1 microcode low, U2 microcode high, U3 74HC138, U4 4011

Commit message: pcb design
Parts:
- added C1: C_Polarized, Capacitor_SMD:CP_Elec_5x5.3, F.Cu at (51.7, 73.0)
- added C2: C, Capacitor_SMD:C_0603_1608Metric, F.Cu at (73.2, 113.7)
- added C3: C, Capacitor_SMD:C_0603_1608Metric, F.Cu at (58.3, 113.7)
- added C4: C, Capacitor_SMD:C_0603_1608Metric, F.Cu at (92.1, 71.3)
- added C5: C, Capacitor_SMD:C_0603_1608Metric, F.Cu at (65.4, 71.3)
Routing:
- net VCC: track 127.8 -> 145.3 mm
