File: circuits/pc-13_microcode/microcode.kicad_sch (KiCad schematic)
At the start: 12 parts, among them J1 Conn_01x05, U1 microcode low, U2 microcode high, U3 74HC138, U4 4011

Commit message: pcb design
Parts:
- added C1: C_Polarized, Capacitor_SMD:CP_Elec_5x5.3, symbol Device:C_Polarized
- added C2, C3, C4, C5: C, Capacitor_SMD:C_0603_1608Metric, symbol Device:C
Connections:
- net GND: now also C1.2, C2.2, C3.2, C4.2, C5.2
- net VCC: now also C1.1, C2.1, C3.1, C4.1, C5.1
