File: circuits/pc-12_sequencer/sequencer.kicad_pcb (KiCad board)
At the start: 2 copper layers, 99.1 x 99.1 mm, 22 parts, among them J1 Screw_Terminal_01x03, U1 74HC273, U10 74HC74, U2 74HC273, U3 74HC273, U4 74LS283, U5 4081, U6 4071, U7 4081, U8 4078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

Commit message: pcb design
Parts:
- added C1: C_Polarized, Capacitor_SMD:CP_Elec_5x5.3, F.Cu at (103.8, 74.3)
- added C2: C, Capacitor_SMD:C_0603_1608Metric, F.Cu at (121.8, 36.8)
- added C3: C, Capacitor_SMD:C_0603_1608Metric, F.Cu at (81.4, 114.3)
- added C4: C, Capacitor_SMD:C_0603_1608Metric, F.Cu at (88.4, 60.3)
- added C5: C, Capacitor_SMD:C_0603_1608Metric, F.Cu at (95.7, 92.7)
Routing:
- net VCC: track 312.3 -> 333.1 mm

Commit message: reworking sequencer PCB
Parts:
- removed D1, D2: D, Diode_THT:D_DO-35_SOD27_P2.54mm_Vertical_KathodeUp
- removed R1: R, Resistor_SMD:R_0603_1608Metric
- added U11: 4011, Package_DIP:DIP-14_W7.62mm, F.Cu at (68.6, 64.1)
- moved C1 52.8 mm to (51.1, 71.8)
- moved U10 12.7 mm to (81.3, 64.1)
- moved U9 12.7 mm to (95.3, 64.1)
- moved C4 12.7 mm to (101.1, 60.3)
- moved C5 9.14 mm to (97.2, 83.7), turned to 90 degrees
Connections:
- U10 pad 10: VCC -> ~{reset}
- U10 pad 13: ~{reset} -> VCC
- U9 pad 1: /interrupt_unit/~{fetch} -> /interrupt_unit/~{interrupt_request}
- U9 pad 10: ~{clock} -> unconnected-(U9-Pad10)
- U9 pad 11: Net-(U10B-D) -> unconnected-(U9-Pad11)
- U9 pad 12: /interrupt_unit/interrupt_allowed -> GND
- U9 pad 13: /interrupt_unit/~{interrupt_request} -> GND
- U9 pad 2: /interrupt_unit/~{fetch} -> /interrupt_unit/interrupt_allowed
- U9 pad 3: /interrupt_unit/fetch -> Net-(U10B-D)
- U9 pad 8: clock -> GND
- U9 pad 9: clock -> GND
Routing:
- net GND: track 34.9 -> 0.00 mm, vias 14 -> 0
- net clock: track 63.2 -> 93.6 mm
- net /~{enint}: track 42.2 -> 61.7 mm
- net /interrupt_unit/~{interrupt}: track 74.8 -> 57.8 mm, vias 0 -> 1
- net ~{reset}: track 164.8 -> 180.7 mm
- net VCC: track 333.1 -> 348.5 mm
- net /interrupt_unit/~{fetch}: track 32.4 -> 45.4 mm, vias 1 -> 0
- net /interrupt_unit/interrupt: track 82.1 -> 70.1 mm, vias 0 -> 1
- net Net-(U10A-~{R}): track 25.8 -> 14.8 mm
- net Net-(U11-Pad1): track 0.00 -> 10.7 mm
- net Net-(U10B-D): track 15.0 -> 6.36 mm
- net /interrupt_unit/load_step: track 62.2 -> 54.3 mm, vias 1 -> 0
- net /interrupt_unit/interrupt_allowed: track 27.7 -> 20.1 mm
- net /interrupt_unit/fetch: track 23.4 -> 17.7 mm
- net /interrupt_unit/~{interrupt_request}: track 59.4 -> 54.3 mm, vias 0 -> 1
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
Commit message: finalize rev. a of pc-12
Connections:
- U9 pad 1: /interrupt_unit/~{interrupt_request} -> Net-(U9-Pad1)
- U9 pad 10: unconnected-(U9-Pad10) -> /interrupt_unit/~{fetch}
- U9 pad 11: unconnected-(U9-Pad11) -> Net-(U9-Pad1)
- U9 pad 12: GND -> /interrupt_unit/~{interrupt_request}
- U9 pad 13: GND -> /interrupt_unit/~{interrupt_request}
- U9 pad 4: /interrupt_unit/~{fetch} -> unconnected-(U9-Pad4)
- U9 pad 5: /interrupt_unit/load_step -> GND
- U9 pad 6: clock -> GND
- U9 pad 8: GND -> clock
- U9 pad 9: GND -> /interrupt_unit/load_step
Routing:
- net GND: track 0.00 -> 27.3 mm, vias 0 -> 7
- net ~{reset}: track 180.7 -> 197.7 mm, vias 2 -> 0
- net Net-(U9-Pad1): track 0.00 -> 13.0 mm
- net /interrupt_unit/interrupt: track 70.1 -> 64.3 mm
- net /interrupt_unit/~{interrupt_request}: track 54.3 -> 59.5 mm
- net /interrupt_unit/load_step: track 54.3 -> 59.5 mm
- net /step_1: track 79.7 -> 76.7 mm
- net /step_0: track 70.4 -> 68.2 mm
- net Net-(U2-D1): track 23.5 -> 25.3 mm
- net Net-(U2-D4): track 31.1 -> 33.0 mm
- net /interrupt_unit/~{fetch}: track 45.4 -> 44.1 mm, vias 0 -> 1
- net Net-(U2-D6): track 31.3 -> 30.6 mm
- net clock: track 93.6 -> 94.0 mm, vias 1 -> 2
